File: spectrePCB/spectrePCB.kicad_pcb (KiCad board)
At the start: 2 copper layers, 282 parts, among them J1 USB_C_Receptacle, SW1 SW_Push, U1 Opamp_Dual_Generic, U2 ADG633YRU, U3 ATmega32U4-AU, U4 ADG633YRU, U5 ADG633YRU, Y1 16MHz

Commit message: placed resistors, added edges, fixing GND net
Parts:
- removed U4, U5: ADG633YRU, Package_SO:TSSOP-20_4.4x6.5mm_P0.65mm
- R1, R2, R3, R4, R5, R6, R7: footprint Resistor_SMD:R_0201_0603Metric -> Resistor_SMD:R_0603_1608Metric
- R10, R11, R12, R13, R14, R15, R16, R17, R18, R19, R20, R21, R22, R23, R24, R25, R26, R27, R28, R29, R30, R31, R32, R33, R34, R35, R36, R37, R38, R39, R40, R41, R42, R43, R44, R45, R46, R47, R48, R49, R50, R51, R52, R53, R54, R55, R56, R57, R58, R59, R60, R61, R62, R63, R64, R65, R66, R67, R68, R69, R70, R71, R72, R8, R9: footprint Resistor_SMD:R_0201_0603Metric -> Resistor_SMD:R_0603_1608Metric; moved to B.Cu
- moved R22 313.3 mm to (14.3, 69.0), turned to 180 degrees
- moved R23 286.9 mm to (38.2, 69.0), turned to 180 degrees
- moved SW1 267.6 mm to (327.0, 29.4)
- moved R60 258.6 mm to (307.2, 107.1), turned to 180 degrees
- moved R48 244.7 mm to (21.3, 107.1), turned to 180 degrees
- moved Y1 238.3 mm to (330.2, 16.7)
- moved R5 236.9 mm to (306.8, 29.8)
- moved R2 236.4 mm to (299.3, 29.8)
- moved R3 235.4 mm to (295.9, 29.8)
- moved R67 235.2 mm to (288.1, 126.2), turned to 180 degrees
- moved R4 234.2 mm to (292.2, 29.8)
- moved R6 233.5 mm to (288.9, 37.3)
- moved R1 231.9 mm to (310.5, 29.8)
- moved C2 231.0 mm to (314.5, 20.2)
- moved C3 231.0 mm to (310.5, 20.2)
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Connections:
- U2 pad 1: (no net) -> Net-(U2-Pad1)
- U2 pad 10: (no net) -> /Switch Matrix/CAPS
- U2 pad 15: (no net) -> /Switch Matrix/L+
- U2 pad 16: (no net) -> +5V
- U2 pad 2: (no net) -> Net-(R72-Pad2)
- U2 pad 6: (no net) -> Net-(U2-Pad6)
- U2 pad 7: (no net) -> ROW0
- U2 pad 8: (no net) -> ROW0
Other:
- board outline added: 335.8 x 131 mm

Commit message: finished routing pcb
Parts:
- D10, D101, D103, D105, D107, D109, D111, D113, D115, D117, D119, D12, D121, D123, D125, D127, D14, D16, D18, D2, D20, D22, D24, D26, D28, D30, D32, D34, D36, D38, D4, D40, D42, D44, D46, D48, D50, D52, D54, D56, D58, D59, D6, D61, D63, D65, D67, D69, D71, D73, D75, D77, D79, D8, D81, D83, D85, D87, D89, D91, D93, D95, D97, D99: moved to B.Cu
- moved D127 156.1 mm to (331.8, 113.5), turned to 270 degrees
- moved R3 151.6 mm to (144.5, 23.0)
- moved D1 149.3 mm to (148.4, 23.0)
- moved D109 147.5 mm to (17.5, 113.5), turned to 270 degrees
- moved SW1 145.9 mm to (181.8, 15.9)
- moved F1 145.3 mm to (152.4, 23.0), turned to 180 degrees
- moved D125 144.1 mm to (312.7, 113.5), turned to 270 degrees
- moved R5 139.5 mm to (167.5, 22.2), turned to 180 degrees
- moved D107 135.3 mm to (312.7, 94.5), turned to 270 degrees
- moved D123 132.8 mm to (293.7, 113.5), turned to 270 degrees
- moved D111 131.9 mm to (41.3, 113.5), turned to 270 degrees
- moved D83 130.6 mm to (27.0, 94.5), turned to 270 degrees
- moved R1 128.9 mm to (181.8, 23.0)
- moved R6 127.9 mm to (161.9, 22.2), turned to 180 degrees
- moved U2 127.8 mm to (148.4, 16.7), turned to 270 degrees
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Connections:
- C1 pad 2: ROW0 -> GND
- C2 pad 2: ROW0 -> GND
- C3 pad 2: ROW0 -> GND
- C4 pad 2: ROW0 -> GND
- C5 pad 2: ROW0 -> GND
- C6 pad 2: ROW0 -> GND
- C7 pad 2: ROW0 -> GND
- D100 pad 1: ROW0 -> GND
- D101 pad 1: ROW0 -> ROW3
- D102 pad 1: ROW0 -> GND
- D103 pad 1: ROW0 -> ROW3
- D104 pad 1: ROW0 -> GND
- D105 pad 1: ROW0 -> ROW3
- D106 pad 1: ROW0 -> GND
- D107 pad 1: ROW0 -> ROW3
- D108 pad 1: ROW0 -> GND
- D109 pad 1: ROW0 -> ROW4
- D11 pad 1: ROW0 -> GND
- D110 pad 1: ROW0 -> GND
- D111 pad 1: ROW0 -> ROW4
- D112 pad 1: ROW0 -> GND
- D113 pad 1: ROW0 -> ROW4
- D114 pad 1: ROW0 -> GND
- D115 pad 1: ROW0 -> ROW4
- D116 pad 1: ROW0 -> GND
- D117 pad 1: ROW0 -> ROW4
- D118 pad 1: ROW0 -> GND
- D119 pad 1: ROW0 -> ROW4
- D120 pad 1: ROW0 -> GND
- D121 pad 1: ROW0 -> ROW4
- D122 pad 1: ROW0 -> GND
- D123 pad 1: ROW0 -> ROW4
- D124 pad 1: ROW0 -> GND
- D125 pad 1: ROW0 -> ROW4
- D126 pad 1: ROW0 -> GND
- D127 pad 1: ROW0 -> ROW4
- D128 pad 1: ROW0 -> GND
- D129 pad 1: ROW0 -> GND
- D13 pad 1: ROW0 -> GND
- D130 pad 1: ROW0 -> GND
- D15 pad 1: ROW0 -> GND
- D17 pad 1: ROW0 -> GND
- D19 pad 1: ROW0 -> GND
- D21 pad 1: ROW0 -> GND
- D23 pad 1: ROW0 -> GND
- D25 pad 1: ROW0 -> GND
- D27 pad 1: ROW0 -> GND
- D29 pad 1: ROW0 -> GND
- D3 pad 1: ROW0 -> GND
- D30 pad 1: ROW0 -> ROW1
- D31 pad 1: ROW0 -> GND
- D32 pad 1: ROW0 -> ROW1
- D33 pad 1: ROW0 -> GND
- D34 pad 1: ROW0 -> ROW1
- D35 pad 1: ROW0 -> GND
- D36 pad 1: ROW0 -> ROW1
- D37 pad 1: ROW0 -> GND
- D38 pad 1: ROW0 -> ROW1
- D39 pad 1: ROW0 -> GND
- D40 pad 1: ROW0 -> ROW1
- D41 pad 1: ROW0 -> GND
- D42 pad 1: ROW0 -> ROW1
- D43 pad 1: ROW0 -> GND
- D44 pad 1: ROW0 -> ROW1
- D45 pad 1: ROW0 -> GND
- D46 pad 1: ROW0 -> ROW1
- D47 pad 1: ROW0 -> GND
- D48 pad 1: ROW0 -> ROW1
- D49 pad 1: ROW0 -> GND
- D5 pad 1: ROW0 -> GND
- D50 pad 1: ROW0 -> ROW1
- D51 pad 1: ROW0 -> GND
- D52 pad 1: ROW0 -> ROW1
- D53 pad 1: ROW0 -> GND
- D54 pad 1: ROW0 -> ROW1
- D55 pad 1: ROW0 -> GND
- D56 pad 1: ROW0 -> ROW1
- D57 pad 1: ROW0 -> GND
- D58 pad 1: ROW0 -> ROW2
- D59 pad 1: ROW0 -> ROW2
- D60 pad 1: ROW0 -> GND
- D61 pad 1: ROW0 -> ROW2
- D62 pad 1: ROW0 -> GND
- D63 pad 1: ROW0 -> ROW2
- D64 pad 1: ROW0 -> GND
- D65 pad 1: ROW0 -> ROW2
- D66 pad 1: ROW0 -> GND
- D67 pad 1: ROW0 -> ROW2
- D68 pad 1: ROW0 -> GND
- D69 pad 1: ROW0 -> ROW2
- D7 pad 1: ROW0 -> GND
- D70 pad 1: ROW0 -> GND
- D71 pad 1: ROW0 -> ROW2
- D72 pad 1: ROW0 -> GND
- D73 pad 1: ROW0 -> ROW2
- D74 pad 1: ROW0 -> GND
- D75 pad 1: ROW0 -> ROW2
- D76 pad 1: ROW0 -> GND
- D77 pad 1: ROW0 -> ROW2
- D78 pad 1: ROW0 -> GND
- D79 pad 1: ROW0 -> ROW2
- D80 pad 1: ROW0 -> GND
- D81 pad 1: ROW0 -> ROW2
- D82 pad 1: ROW0 -> GND
- D83 pad 1: ROW0 -> ROW3
- D84 pad 1: ROW0 -> GND
- D85 pad 1: ROW0 -> ROW3
- D86 pad 1: ROW0 -> GND
- D87 pad 1: ROW0 -> ROW3
- D88 pad 1: ROW0 -> GND
- D89 pad 1: ROW0 -> ROW3
- D9 pad 1: ROW0 -> GND
- D90 pad 1: ROW0 -> GND
- D91 pad 1: ROW0 -> ROW3
- D92 pad 1: ROW0 -> GND
- D93 pad 1: ROW0 -> ROW3
- D94 pad 1: ROW0 -> GND
- D95 pad 1: ROW0 -> ROW3
- D96 pad 1: ROW0 -> GND
- D97 pad 1: ROW0 -> ROW3
- D98 pad 1: ROW0 -> GND
- D99 pad 1: ROW0 -> ROW3
- J1 pad A1: ROW0 -> GND
- J1 pad A10: Net-(J1-PadA10) -> (no net)
- J1 pad A11: Net-(J1-PadA11) -> (no net)
- J1 pad A12: ROW0 -> GND
- J1 pad A2: Net-(J1-PadA2) -> (no net)
- J1 pad A3: Net-(J1-PadA3) -> (no net)
- J1 pad A8: Net-(J1-PadA8) -> (no net)
- J1 pad B1: ROW0 -> GND
- J1 pad B10: Net-(J1-PadB10) -> (no net)
- J1 pad B11: Net-(J1-PadB11) -> (no net)
- J1 pad B12: ROW0 -> GND
- J1 pad B2: Net-(J1-PadB2) -> (no net)
- J1 pad B3: Net-(J1-PadB3) -> (no net)
- J1 pad B8: Net-(J1-PadB8) -> (no net)
- J1 pad S1: ROW0 -> GND
- R19 pad 1: Net-(R19-Pad1) -> /Switch Matrix/L+
- R3 pad 1: ROW0 -> GND
- R5 pad 1: ROW0 -> GND
- R6 pad 1: ROW0 -> GND
- R7 pad 1: ROW0 -> GND
- SW1 pad 1: ROW0 -> GND
- U1 pad 4: ROW0 -> GND
- U2 pad 1: Net-(U2-Pad1) -> (no net)
- U2 pad 13: Net-(U2-Pad13) -> (no net)
- U2 pad 15: /Switch Matrix/L+ -> +5V
- U2 pad 2: Net-(R72-Pad2) -> Net-(R71-Pad2)
- U2 pad 3: Net-(R71-Pad2) -> Net-(R72-Pad2)
- U2 pad 4: +5V -> /Switch Matrix/L+
- U2 pad 5: Net-(U2-Pad5) -> (no net)
- U2 pad 6: Net-(U2-Pad6) -> (no net)
- U2 pad 7: ROW0 -> GND
- U2 pad 8: ROW0 -> GND
- U3 pad 10: MOSI -> (no net)
- U3 pad 11: MISO -> (no net)
- U3 pad 15: ROW0 -> GND
- U3 pad 18: ROW0 -> ROW1
- U3 pad 19: ROW0 -> ROW2
- U3 pad 20: ROW0 -> ROW3
- U3 pad 21: ROW0 -> ROW4
- U3 pad 22: COL14 -> COL13
- U3 pad 23: ROW0 -> GND
- U3 pad 25: COL13 -> COL14
- U3 pad 26: COL12 -> COL0
- U3 pad 27: COL11 -> COL1
- U3 pad 28: COL10 -> COL2
- U3 pad 29: COL9 -> COL3
- U3 pad 30: COL8 -> COL4
- U3 pad 31: COL7 -> COL5
- U3 pad 35: ROW0 -> GND
- U3 pad 36: COL5 -> COL7
- U3 pad 37: COL4 -> COL8
- U3 pad 38: COL3 -> COL9
- U3 pad 39: COL2 -> COL10
- U3 pad 40: COL1 -> COL11
- U3 pad 41: COL0 -> COL12
- U3 pad 42: Net-(U3-Pad42) -> (no net)
- U3 pad 43: ROW0 -> GND
- U3 pad 5: ROW0 -> GND
- U3 pad 8: CAPS -> (no net)
- U3 pad 9: SCK -> (no net)
- Y1 pad 2: ROW0 -> GND
- Y1 pad 4: ROW0 -> GND
Routing:
- net /Switch Matrix/L+: track 0.00 -> 1728.6 mm, vias 0 -> 10
- net COL0: track 0.00 -> 459.0 mm
- net COL1: track 0.00 -> 440.1 mm
- net COL2: track 0.00 -> 415.4 mm
- net ROW4: track 0.00 -> 382.5 mm, vias 0 -> 5
- net COL3: track 0.00 -> 373.6 mm
- net COL5: track 0.00 -> 356.5 mm
- net COL4: track 0.00 -> 351.6 mm
- net GND: track 0.00 -> 348.7 mm, vias 0 -> 77
- net ROW3: track 0.00 -> 340.2 mm, vias 0 -> 5
- net COL6: track 0.00 -> 310.0 mm
- net ROW2: track 0.00 -> 309.0 mm, vias 0 -> 5
- net ROW0: track 0.00 -> 306.8 mm, vias 0 -> 3
- net ROW1: track 0.00 -> 294.3 mm, vias 0 -> 3
- net COL7: track 0.00 -> 282.6 mm
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- added copper zone on B.Cu, net GND
Other:
- board size 335.8 x 131 mm -> 335.8 x 120.7 mm
- net class Default: clearance 0.2 -> 0.1524; trace_width 0.25 -> 0.2032; via_dia 0.8 -> 0.6858; via_drill 0.4 -> 0.3048
- net class Power added: clearance 0.1524, trace_width 0.381, via_dia 0.6858, via_drill 0.3048
- rule pad_to_mask_clearance: 0 -> 0.00129
- rule trace_clearance: 0.2 -> 0.1524
- rule trace_min: 0.2 -> 0.1524
- rule via_min_drill: 0.3 -> 0.254
- rule via_min_size: 0.4 -> 0.508
